File: Project 2/Project 2.kicad_pcb (KiCad board)
At the start: 2 copper layers, 32 parts, among them J1 Upload_Pins, J4 Servo_1, J5 Bluetooth, J6 LCD, J7 Servo_2, Q1 IRF540N, Q2 IRF540N, Q3 IRF540N, Q4 IRF540N, Q5 IRF540N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

Commit message: initial PCB design
Parts:
- added C1: 1nF, Capacitor_THT:C_Disc_D3.0mm_W2.0mm_P2.50mm, F.Cu at (173.9, 57.7)
- added C10: 22pF, Capacitor_THT:C_Disc_D3.0mm_W2.0mm_P2.50mm, F.Cu at (150.2, 82.3)
- added C11: 22pF, Capacitor_THT:C_Disc_D3.0mm_W2.0mm_P2.50mm, F.Cu at (150.2, 86.6)
- added C12: 1uF, Capacitor_THT:C_Radial_D5.0mm_H11.0mm_P2.00mm, F.Cu at (115.1, 142.8)
- added C13: 1uF, Capacitor_THT:C_Radial_D5.0mm_H11.0mm_P2.00mm, F.Cu at (137.9, 143.0)
- added C14: 1uF, Capacitor_THT:C_Radial_D5.0mm_H11.0mm_P2.00mm, F.Cu at (122.6, 142.8)
- added C15: 1uF, Capacitor_THT:C_Radial_D5.0mm_H11.0mm_P2.00mm, F.Cu at (88.6, 82.8)
- added C16: 1nF, Capacitor_THT:C_Disc_D3.0mm_W2.0mm_P2.50mm, F.Cu at (94.3, 108.0)
- added C2: 100pF, Capacitor_THT:C_Disc_D3.0mm_W2.0mm_P2.50mm, F.Cu at (173.9, 65.8)
- added C3: 10uF, Capacitor_THT:C_Radial_D5.0mm_H11.0mm_P2.00mm, F.Cu at (100.9, 119.4)
- added C4: 10uF, Capacitor_THT:C_Radial_D5.0mm_H11.0mm_P2.00mm, F.Cu at (139.7, 128.8)
- added C5: 10uF, Capacitor_THT:C_Radial_D5.0mm_H11.0mm_P2.00mm, F.Cu at (124.0, 128.8)
- added C6: 10uF, Capacitor_THT:C_Radial_D5.0mm_H11.0mm_P2.00mm, F.Cu at (108.5, 128.8)
- added C7: 1uF, Capacitor_THT:C_Radial_D5.0mm_H11.0mm_P2.00mm, F.Cu at (145.3, 143.0)
- added C8: 1uF, Capacitor_THT:C_Radial_D5.0mm_H11.0mm_P2.00mm, F.Cu at (129.9, 142.9)
- added C9: 1uF, Capacitor_THT:C_Radial_D5.0mm_H11.0mm_P2.00mm, F.Cu at (107.7, 142.7)
- added G***: LOGO, LOGO, F.Cu at (150.6, 118.9)
- added G***: LOGO, LOGO, F.Cu at (151.4, 105.4)
- added J2: Jack-DC, Connector_BarrelJack:BarrelJack_GCT_DCJ200-10-A_Horizontal, F.Cu at (187.7, 91.9)
- added J3: BLDC_Output, TerminalBlock:TerminalBlock_Altech_AK300-3_P5.00mm, F.Cu at (190.8, 118.4)
- added R17: 10k, Resistor_THT:R_Axial_DIN0207_L6.3mm_D2.5mm_P7.62mm_Horizontal, F.Cu at (97.8, 111.5)
- added R18: 4.7k, Resistor_THT:R_Axial_DIN0207_L6.3mm_D2.5mm_P7.62mm_Horizontal, F.Cu at (92.5, 94.5)
- added R19: 220, Resistor_THT:R_Axial_DIN0207_L6.3mm_D2.5mm_P7.62mm_Horizontal, F.Cu at (97.0, 91.9)
- added R20: 220, Resistor_THT:R_Axial_DIN0207_L6.3mm_D2.5mm_P7.62mm_Horizontal, F.Cu at (97.3, 87.1)
- added RV1: 5k, Potentiometer_THT:Potentiometer_Bourns_3386P_Vertical, F.Cu at (163.3, 85.9)
- added SW1: Reset_Button, Button_Switch_THT:SW_PUSH_6mm_H4.3mm, F.Cu at (147.1, 93.0)
- added U3: IR2104, Package_SO:SOIC-8_3.9x4.9mm_P1.27mm, F.Cu at (139.7, 136.9)
- added U4: IR2104, Package_SO:SOIC-8_3.9x4.9mm_P1.27mm, F.Cu at (124.2, 136.9)
- added U5: IR2104, Package_SO:SOIC-8_3.9x4.9mm_P1.27mm, F.Cu at (108.7, 136.9)
- added U6: mystery_uart_thing, Package_SO:SOP-16_3.9x9.9mm_P1.27mm, F.Cu at (96.8, 100.8)
- added Y1: Crystal, Crystal:Crystal_AT310_D3.0mm_L10.0mm_Vertical, F.Cu at (143.3, 83.1)
- J1: value Upload_Pins -> USB_B; footprint Connector_PinSocket_2.54mm:PinSocket_1x05_P2.54mm_Vertical -> Connector_USB:USB_B_Lumberg_2411_02_Horizontal
- J6: footprint Connector_PinSocket_2.54mm:PinSocket_1x16_P2.54mm_Vertical -> Display:WC1602A
- moved R16 97.0 mm to (97.3, 82.3)
- moved J1 88.5 mm to (94.7, 119.4), turned to 180 degrees
- moved J5 83.3 mm to (86.8, 104.1), turned to 180 degrees
- moved D3 82.3 mm to (116.6, 138.4), turned to 90 degrees
- moved R3 68.5 mm to (180.1, 144.8), turned to 90 degrees
- moved J6 66.9 mm to (93.5, 45.4)
- moved J7 65.8 mm to (187.5, 130.6), turned to 90 degrees
- moved R2 65.2 mm to (175.3, 144.8), turned to 90 degrees
- moved R11 62.3 mm to (160.8, 126.5), turned to -90 degrees
- moved Q6 61.8 mm to (173.0, 129.5)
- moved R1 57.4 mm to (170.4, 144.8), turned to 90 degrees
- moved Q3 53.1 mm to (173.0, 105.2)
- moved R10 51.7 mm to (159.3, 119.4)
- moved D1 50.1 mm to (146.6, 138.7), turned to 90 degrees
- moved R4 49.2 mm to (165.6, 126.5), turned to -90 degrees
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Connections:
- J1 pad 1: GND -> +5V
- J1 pad 2: +5V -> D-
- J1 pad 3: Tx -> D+
- J1 pad 4: Rx -> GND
- J1 pad 5: Reset -> unconnected-(J1-Pad5)
- J6 pad 11: 26 -> 25
- J6 pad 12: GND -> 24
- J6 pad 13: 27 -> 23
- J6 pad 14: Net-(J6-Pad14) -> 22
- J6 pad 15: +5V -> Net-(J6-Pad15)
- J6 pad 2: Net-(J6-Pad2) -> +5V
- J6 pad 3: 22 -> Net-(J6-Pad3)
- J6 pad 4: 23 -> 27
- J6 pad 5: 24 -> GND
- J6 pad 6: 25 -> 26
- R16 pad 2: Net-(J6-Pad2) -> Net-(J6-Pad15)
Routing:
- net +5V: track 0.00 -> 124.6 mm, vias 0 -> 2
- net Net-(J6-Pad3): track 0.00 -> 94.1 mm, vias 0 -> 2
- net 13: track 0.00 -> 91.0 mm, vias 0 -> 1
- net 8: track 0.00 -> 89.1 mm, vias 0 -> 1
- net Net-(J3-Pad2): track 0.00 -> 88.4 mm, vias 0 -> 4
- net 12: track 0.00 -> 84.8 mm, vias 0 -> 7
- net Net-(J3-Pad1): track 0.00 -> 84.2 mm, vias 0 -> 2
- net Net-(J6-Pad15): track 0.00 -> 83.8 mm, vias 0 -> 3
- net 7: track 0.00 -> 83.7 mm, vias 0 -> 4
- net 23: track 0.00 -> 83.5 mm, vias 0 -> 2
- net 22: track 0.00 -> 82.2 mm, vias 0 -> 3
- net 25: track 0.00 -> 80.9 mm, vias 0 -> 2
- net 6: track 0.00 -> 80.8 mm, vias 0 -> 2
- net 24: track 0.00 -> 77.7 mm, vias 0 -> 3
- net Reset: track 0.00 -> 73.5 mm, vias 0 -> 2
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- added copper zone on F.Cu, net +12V
- added copper zone on F.Cu, net +5V
- added copper zone on B.Cu, net GND
Other:
- board outline added: 114.6 x 108.5 mm
- board text added: "According to all known laws of aviation, there is no way that a bee should be able to fly. Its wings are too small to get its fat little body off the ground. The bee, of course, flies anyway. Because bees don't care what humans think is impossible.{dblquote} SEQ. 75 - {dblquote}INTRO TO BARRY{dblquote} INT. BENSON HOUSE - DAY ANGLE ON: Sneakers on the ground. Camera PANS UP to reveal BARRY BENSON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"
- board text added: "RC Plane PCB V1.0 EE 333 Project 2 Austin Beinder and Jonah Frosch"

Commit message: added current pcb
Parts:
- removed the G*** at (150.6, 118.9)
- removed the G*** at (151.4, 105.4)
- added D4: Bluetooth, LED_THT:LED_D3.0mm, F.Cu at (74.3, 77.9)
- added D5: Power LED, LED_THT:LED_D3.0mm, F.Cu at (74.3, 70.3)
- added D6: Serial, LED_THT:LED_D3.0mm, F.Cu at (74.3, 62.6)
- added G***: LOGO, LOGO, F.Cu at (123.4, 119.4)
- added G***: LOGO, LOGO, F.Cu at (197.9, 131.3)
- added G***: LOGO, LOGO, F.Cu at (150.9, 120.9)
- added G***: LOGO, LOGO, F.Cu at (207.0, 44.5)
- added G***: LOGO, LOGO, F.Cu at (196.1, 36.8)
- added G***: LOGO, LOGO, F.Cu at (194.8, 46.7)
- added H1: MountingHole, MountingHole:MountingHole_5mm_Pad, F.Cu at (73.4, 135.4)
- added H2: MountingHole, MountingHole:MountingHole_5mm_Pad, F.Cu at (212.6, 135.4)
- added H3: MountingHole, MountingHole:MountingHole_5mm_Pad, F.Cu at (212.6, 35.1)
- added H4: MountingHole, MountingHole:MountingHole_5mm_Pad, F.Cu at (73.4, 35.1)
- added R21: 0, Resistor_THT:R_Axial_DIN0207_L6.3mm_D2.5mm_P7.62mm_Horizontal, F.Cu at (161.0, 77.3)
- added R22: 0, Resistor_THT:R_Axial_DIN0207_L6.3mm_D2.5mm_P7.62mm_Horizontal, F.Cu at (161.0, 82.1)
- added R23: 0, Resistor_THT:R_Axial_DIN0207_L6.3mm_D2.5mm_P7.62mm_Horizontal, F.Cu at (161.0, 86.9)
- added R24: 0, Resistor_THT:R_Axial_DIN0207_L6.3mm_D2.5mm_P7.62mm_Horizontal, F.Cu at (161.0, 91.8)
- added R25: 0, Resistor_THT:R_Axial_DIN0207_L6.3mm_D2.5mm_P7.62mm_Horizontal, F.Cu at (161.0, 96.6)
- added R26: 0, Resistor_THT:R_Axial_DIN0207_L6.3mm_D2.5mm_P7.62mm_Horizontal, F.Cu at (161.0, 101.4)
- added R27: 0, Resistor_THT:R_Axial_DIN0207_L6.3mm_D2.5mm_P7.62mm_Horizontal, F.Cu at (193.5, 55.1)
- added R28: 0, Resistor_THT:R_Axial_DIN0207_L6.3mm_D2.5mm_P7.62mm_Horizontal, F.Cu at (193.5, 61.0)
- added R29: 1k, Resistor_THT:R_Axial_DIN0207_L6.3mm_D2.5mm_P7.62mm_Horizontal, F.Cu at (84.5, 84.7)
- added R30: 1k, Resistor_THT:R_Axial_DIN0207_L6.3mm_D2.5mm_P7.62mm_Horizontal, F.Cu at (79.6, 84.7)
- added R31: 1k, Resistor_THT:R_Axial_DIN0207_L6.3mm_D2.5mm_P7.62mm_Horizontal, F.Cu at (74.8, 84.7)
- J3: footprint TerminalBlock:TerminalBlock_Altech_AK300-3_P5.00mm -> Connector_PinSocket_2.54mm:PinSocket_1x03_P2.54mm_Vertical
- moved J2 105.9 mm to (82.2, 100.9), turned to -90 degrees
- moved U2 105.3 mm to (94.5, 120.2), turned to 180 degrees
- moved C2 98.5 mm to (88.6, 115.1)
- moved C1 97.6 mm to (95.0, 115.1), turned to 90 degrees
- moved C9 86.6 mm to (188.7, 112.3), turned to 0 degrees
- moved C14 84.5 mm to (188.7, 90.2), turned to 0 degrees
- moved J4 83.5 mm to (212.1, 61.7), turned to -90 degrees
- moved C12 82.8 mm to (188.7, 105.0), turned to 0 degrees
- moved RV1 80.5 mm to (99.3, 37.1)
- moved C7 80.3 mm to (188.7, 75.5), turned to 0 degrees
- moved J7 79.4 mm to (212.3, 55.1), turned to -90 degrees
- moved U5 78.8 mm to (182.4, 109.0), turned to 0 degrees
- moved C13 78.7 mm to (188.7, 82.9), turned to 0 degrees
- moved D3 78.4 mm to (185.9, 101.9), turned to 180 degrees
- moved D1 77.1 mm to (185.7, 72.2), turned to 180 degrees
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Connections:
- J3 pad 1: Net-(J3-Pad1) -> Net-(C13-Pad2)
- J3 pad 2: Net-(J3-Pad2) -> Net-(C14-Pad2)
- J3 pad 3: Net-(J3-Pad3) -> Net-(C12-Pad2)
- J4 pad 3: 8 -> Net-(J4-Pad3)
- J7 pad 3: 13 -> Net-(J7-Pad3)
- Q1 pad 3: Net-(J3-Pad1) -> Net-(C13-Pad2)
- Q2 pad 2: Net-(J3-Pad1) -> Net-(C13-Pad2)
- Q3 pad 3: Net-(J3-Pad2) -> Net-(C14-Pad2)
- Q4 pad 2: Net-(J3-Pad2) -> Net-(C14-Pad2)
- Q5 pad 3: Net-(J3-Pad3) -> Net-(C12-Pad2)
- Q6 pad 2: Net-(J3-Pad3) -> Net-(C12-Pad2)
- R1 pad 1: 6 -> pin 4
- R1 pad 2: 7 -> A4
- R13 pad 1: 7 -> A4
- R13 pad 2: Net-(J3-Pad1) -> Net-(C13-Pad2)
- R14 pad 2: Net-(J3-Pad2) -> Net-(C14-Pad2)
- R15 pad 2: Net-(J3-Pad3) -> Net-(C12-Pad2)
- R2 pad 1: 6 -> pin 4
- R3 pad 1: 6 -> pin 4
- R4 pad 1: 7 -> A4
- U1 pad 15: 6 -> unconnected-(U1-Pad15)
- U1 pad 16: 7 -> unconnected-(U1-Pad16)
- U1 pad 17: 8 -> unconnected-(U1-Pad17)
- U1 pad 24: unconnected-(U1-Pad24) -> 11
- U1 pad 4: unconnected-(U1-Pad4) -> pin 4
- U1 pad 45: Rx1 -> Tx1
- U1 pad 46: Tx1 -> Rx1
- U1 pad 93: unconnected-(U1-Pad93) -> A4
- U3 pad 2: 5 -> Net-(R21-Pad2)
- U3 pad 3: 12 -> Net-(R22-Pad2)
- U4 pad 2: 4 -> Net-(R23-Pad2)
- U4 pad 3: 10 -> Net-(R24-Pad2)
- U5 pad 2: 3 -> Net-(R25-Pad2)
- U5 pad 3: 9 -> Net-(R26-Pad2)
Routing:
- net Net-(C13-Pad2): track 14.7 -> 119.8 mm, vias 0 -> 3
- net +5V: track 124.6 -> 34.3 mm, vias 2 -> 4
- net 8: track 89.1 -> 0.00 mm, vias 1 -> 0
- net Net-(J3-Pad2): track 88.4 -> 0.00 mm, vias 4 -> 0
- net Net-(J3-Pad1): track 84.2 -> 0.00 mm, vias 2 -> 0
- net 7: track 83.7 -> 0.00 mm, vias 4 -> 0
- net Net-(C14-Pad2): track 14.4 -> 96.3 mm, vias 0 -> 2
- net 6: track 80.8 -> 0.00 mm, vias 2 -> 0
- net A4: track 0.00 -> 73.9 mm
- net 11: track 0.00 -> 73.6 mm, vias 0 -> 1
- net Net-(J6-Pad3): track 94.1 -> 25.0 mm, vias 2 -> 0
- net pin 4: track 0.00 -> 64.6 mm, vias 0 -> 1
- net Net-(R9-Pad1): track 66.3 -> 11.6 mm, vias 2 -> 1
- net Net-(R7-Pad1): track 65.0 -> 11.0 mm
- net Net-(J3-Pad3): track 53.4 -> 0.00 mm
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Other:
- board size 114.6 x 108.5 mm -> 149.9 x 111 mm
- board text added: "RC Plane that has to be plugged into the wall V1.2 Section 1 Group 2: By Austin Beinder and Jonah Frosch EE 333 Project 2"
- board text removed: "According to all known laws of aviation, there is no way that a bee should be able to fly. Its wings are too small to get its fat little body off the ground. The bee, of course, flies anyway. Because bees don't care what humans think is impossible.{dblquote} SEQ. 75 - {dblquote}INTRO TO BARRY{dblquote} INT. BENSON HOUSE - DAY ANGLE ON: Sneakers on the ground. Camera PANS UP to reveal BARRY BENSON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"
- board text removed: "RC Plane PCB V1.0 EE 333 Project 2 Austin Beinder and Jonah Frosch"
