File: Project 2/Project 2.kicad_sch (KiCad schematic)
At the start: 61 parts, among them J1 USB_B, J2 Jack-DC, J3 BLDC_Output, J4 Servo_1, J5 Bluetooth, J6 LCD, J7 Servo_2, Q1 IRF540N, Q2 IRF540N, Q3 IRF540N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

Commit message: added current pcb
Parts:
- added D4: Bluetooth, LED_THT:LED_D3.0mm, symbol Device:LED
- added D5: Power LED, LED_THT:LED_D3.0mm, symbol Device:LED
- added D6: Serial, LED_THT:LED_D3.0mm, symbol Device:LED
- added H1, H2, H3, H4: MountingHole, MountingHole:MountingHole_5mm_Pad, symbol Mechanical:MountingHole
- added R21, R22, R23, R24, R25, R26, R27, R28: 0, Resistor_THT:R_Axial_DIN0207_L6.3mm_D2.5mm_P7.62mm_Horizontal, symbol Device:R
- added R29, R30, R31: 1k, Resistor_THT:R_Axial_DIN0207_L6.3mm_D2.5mm_P7.62mm_Horizontal, symbol Device:R
- J3: footprint TerminalBlock:TerminalBlock_Altech_AK300-3_P5.00mm -> Connector_PinSocket_2.54mm:PinSocket_1x03_P2.54mm_Vertical
Connections:
- net +5V: now also D5.2 (A)
- net 10: now also R24.1; no longer U4.3 (~{SD})
- net 11: now also U1.24 (PB5), R22.1
- net 12: now also R28.1; no longer U3.3 (~{SD})
- net 13: now also R27.1; no longer J7.3 (Pin_3)
- net 3: now also R25.1; no longer U5.2 (IN)
- net 4: now also R23.1; no longer U4.2 (IN)
- net 5: now also R21.1; no longer U3.2 (IN)
- net 8: no longer J4.3 (Pin_3), U1.17 (PH5)
- net 9: now also R26.1; no longer U5.3 (~{SD})
- net GND: now also R29.2, R30.2, R31.2
- net Rx1: now also U1.46 (PD3); no longer U1.45 (PD2)
- net Tx: now also D6.2 (A)
- net Tx1: now also U1.45 (PD2), D4.2 (A); no longer U1.46 (PD3)
- net at C13.2, C7.2, U3.6 (VS): now also J3.1 (Pin_1), Q1.3 (S), Q2.2 (D), R13.2
- net at C12.2, C9.2, U5.6 (VS): now also J3.3 (Pin_3), Q5.3 (S), Q6.2 (D), R15.2
- net at J3.2 (Pin_2), Q3.3 (S), Q4.2 (D)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: now also C14.2, C8.2, U4.6 (VS)
- net pin 4: now reaches U1.4 (PE2)
- net pin 4: now also R1.1, R2.1, R3.1
- net A4: now reaches U1.93 (PF4)
- net A4: now also R1.2, R13.1, R4.1
- removed net 6: R1.1, R2.1, R3.1, U1.15 (PH3)
- removed net 7: R1.2, R13.1, R4.1, U1.16 (PH4)
- new net: R25.2, U5.2 (IN)
- new net: R26.2, U5.3 (~{SD})
- new net: D5.1 (K), R30.1
- new net: D6.1 (K), R31.1
- new net: R23.2, U4.2 (IN)
- new net: R24.2, U4.3 (~{SD})
- new net: J4.3 (Pin_3), R28.2
- new net: R22.2, U3.3 (~{SD})
- new net: R21.2, U3.2 (IN)
- new net: J7.3 (Pin_3), R27.2
- new net: D4.1 (K), R29.1
Other:
- moved on the sheet: C15, C16, C3, R18, R19, R20, U6
